File: OPAMP.kicad_pcb (KiCad board)
At the start: 2 copper layers, 33 x 23 mm, 49 parts, among them J1 GH125-S02CCA-00, J2 GH125-S06DCA-00, J3 GH125-S03DCA-00, SW1 DSHP02TSGET, U1 ADG704BRMZ-REEL, U2 AD8421BRZ-RL, U3 OPA2197QDGKRQ1, U4 REF2030AIDDCR

Commit message: remake
Parts:
- removed J2: GH125-S06DCA-00, kicad_api_lib:GH125-S06DCA-00
- added J4: GH125-S02CCA-00, kicad_api_lib:GH125-S02CCA-00, F.Cu at (121.6, 85.0)
- C1, C10, C11, C12, C13, C14, C15, C16, C17, C18, C2, C3, C4, C5, C6, C7, C8, C9, R1, R10, R13, R14, R15, R16, R17, R18, R19, R2, R20, R3, R4, R5, R6, R7, R8, R9: footprint Capacitor_SMD:C_0201_0603Metric -> Capacitor_SMD:C_0603_1608Metric
- R11, R12: footprint Capacitor_SMD:C_0201_0603Metric -> Capacitor_SMD:C_0603_1608Metric; moved to F.Cu
- moved R6 113.9 mm to (158.8, 83.2), turned to -90 degrees
- moved R9 113.6 mm to (157.2, 83.2), turned to -90 degrees
- moved R8 111.8 mm to (156.8, 85.5), turned to 180 degrees
- moved R7 110.8 mm to (156.8, 87.1), turned to 180 degrees
- moved R10 110.3 mm to (154.9, 82.4)
- moved R5 108.5 mm to (154.9, 83.9)
- moved R4 107.2 mm to (151.8, 82.3), turned to 0 degrees
- moved R3 106.0 mm to (151.8, 84.0), turned to 0 degrees
- moved U1 102.3 mm to (151.6, 86.8), turned to 90 degrees
- moved R13 98.4 mm to (151.8, 80.8)
- moved J3 95.8 mm to (160.3, 90.3)
- moved SW1 95.7 mm to (145.2, 83.1), turned to -90 degrees
- moved R14 94.2 mm to (150.5, 89.8)
- moved R18 93.8 mm to (154.6, 93.7), turned to 90 degrees
- moved C14 92.8 mm to (154.6, 90.6), turned to -90 degrees
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Connections:
- J1 pad 1: /COIL_RAW_P -> /COIL_RAW_N
- J1 pad 2: /COIL_RAW_N -> /COIL_RAW_P
Routing:
- net /AGND_SHIELD: track 66.3 -> 109.6 mm
- net /RG_A: track 10.4 -> 32.8 mm, vias 0 -> 2
- net /RG_B: track 8.46 -> 28.4 mm, vias 0 -> 2
- net +5VA: track 40.0 -> 55.6 mm, vias 2 -> 6
- net /BIAS_1V5: track 27.1 -> 39.2 mm, vias 3 -> 0
- net /+5VIN: track 11.6 -> 0.00 mm
- net /BIAS_FILT: track 9.54 -> 1.90 mm
- net Net-(U1-EN): track 13.8 -> 7.37 mm
- net Net-(U1-A0): track 12.9 -> 7.45 mm
- net Net-(U1-S1): track 2.22 -> 7.17 mm
- net Net-(SW1-B2): track 7.30 -> 2.44 mm, vias 0 -> 2
- net Net-(U4-EN): track 6.80 -> 1.95 mm
- net /VREF_3V0: track 3.50 -> 0.00 mm, vias 2 -> 0
- net Net-(SW1-B1): track 4.90 -> 2.02 mm
- net /VOUT_RAW: track 10.4 -> 12.8 mm, vias 2 -> 0
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- added copper zone on F.Cu, net /BIAS_RAW
- added copper zone on F.Cu, net /VREF_3V0
- removed copper zone on F.Cu, net /AGND_SHIELD
- removed copper zone on F.Cu, net /COIL_FILT_N
- removed copper zone on F.Cu, net /COIL_FILT_P
- removed copper zone on F.Cu, net /RG_A
Other:
- board size 33 x 23 mm -> 46 x 17 mm
