File: OPAMP.kicad_sch (KiCad schematic)
At the start: 49 parts, among them J1 GH125-S02CCA-00, J2 GH125-S06DCA-00, J3 GH125-S03DCA-00, SW1 DSHP02TSGET, U1 ADG704BRMZ-REEL, U2 AD8421BRZ-RL, U3 OPA2197QDGKRQ1, U4 REF2030AIDDCR

Commit message: update
Parts:
- R11, R12: value 1M -> 100K
- R3, R4: value 100 -> 0
Changed lines of the file:
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@@
 			)
 		)
-		(property "Value" "100"
+		(property "Value" "0"
 			(at 59.69 166.37 90)
 			(effects
@@
 			)
 		)
-		(property "Value" "100"
+		(property "Value" "0"
 			(at 59.69 168.91 90)
 			(effects
@@
 			)
 		)
-		(property "Value" "1M"
+		(property "Value" "100K"
 			(at 77.47 122.682 90)
 			(effects
@@
 			)
 		)
-		(property "Value" "1M"
+		(property "Value" "100K"
 			(at 77.47 130.556 90)
 			(effects

Commit message: update
Parts:
- C11: value 1uF -> 4.7uF
- C12: value 330pF -> 47nF
- R14: value 330K -> 68K
- R15: value 4.99K -> 1K
- R18: value 143K -> 28.7K
Changed lines of the file:
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@@
 			)
 		)
-		(property "Value" "143K"
+		(property "Value" "28.7K"
 			(at 196.85 115.57 90)
 			(effects
@@
 			)
 		)
-		(property "Value" "330pF"
+		(property "Value" "47nF"
 			(at 197.104 108.712 90)
 			(effects
@@
 			)
 		)
-		(property "Value" "4.99K"
+		(property "Value" "1K"
 			(at 163.83 117.602 90)
 			(effects
@@
 			)
 		)
-		(property "Value" "1uF"
+		(property "Value" "4.7uF"
 			(at 160.02 90.932 90)
 			(effects
@@
 			)
 		)
-		(property "Value" "330K"
+		(property "Value" "68K"
 			(at 160.02 101.346 90)
 			(effects

Commit message: Layout
Connections:
- net COIL_N_FILT renamed COIL_FILT_N
- net COIL_N_RAW renamed COIL_RAW_N
- net COIL_P_FILT renamed COIL_FILT_P
- net COIL_P_RAW renamed COIL_RAW_P
Changed lines of the file:
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@@
 		)
 	)
-	(label "COIL_P_FILT"
+	(label "COIL_FILT_P"
 		(at 72.39 88.9 180)
 		(effects
@@
 		)
 	)
-	(label "COIL_P_RAW"
+	(label "COIL_RAW_P"
 		(at 27.94 104.14 180)
 		(effects
@@
 		)
 	)
-	(label "COIL_N_RAW"
+	(label "COIL_RAW_N"
 		(at 27.94 113.03 180)
 		(effects
@@
 		)
 	)
-	(label "COIL_P_FILT"
+	(label "COIL_FILT_P"
 		(at 35.56 86.36 0)
 		(effects
@@
 		)
 	)
-	(label "COIL_P_FILT"
+	(label "COIL_FILT_P"
 		(at 73.66 120.65 180)
 		(effects
@@
 		)
 	)
-	(label "COIL_P_RAW"
+	(label "COIL_RAW_P"
 		(at 27.94 86.36 180)
 		(effects
@@
 		)
 	)
-	(label "COIL_P_FILT"
+	(label "COIL_FILT_P"
 		(at 27.94 120.65 180)
 		(effects
@@
 		)
 	)
-	(label "COIL_N_FILT"
+	(label "COIL_FILT_N"
 		(at 72.39 91.44 180)
 		(effects
@@
 		)
 	)
-	(label "COIL_N_FILT"
+	(label "COIL_FILT_N"
 		(at 73.66 128.27 180)
 		(effects
@@
 		)
 	)
-	(label "COIL_N_RAW"
+	(label "COIL_RAW_N"
 		(at 34.29 46.99 0)
 		(effects
@@
 		)
 	)
-	(label "COIL_N_RAW"
+	(label "COIL_RAW_N"
 		(at 27.94 95.25 180)
 		(effects
@@
 		)
 	)
-	(label "COIL_N_FILT"
+	(label "COIL_FILT_N"
 		(at 35.56 95.25 0)
 		(effects
@@
 		)
 	)
-	(label "COIL_N_FILT"
+	(label "COIL_FILT_N"
 		(at 27.94 128.27 180)
 		(effects
@@
 		)
 	)
-	(label "COIL_P_RAW"
+	(label "COIL_RAW_P"
 		(at 31.75 46.99 180)
 		(effects

Commit message: update
Connections:
- net AGND: no longer D1.2, D2.2
- net AGND_SHIELD: now also D1.2, D2.2
Changed lines of the file:
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@@
 		)
 	)
-	(label "AGND"
+	(label "AGND_SHIELD"
 		(at 48.26 113.03 0)
 		(effects
@@
 		)
 	)
-	(label "AGND"
+	(label "AGND_SHIELD"
 		(at 48.26 104.14 0)
 		(effects

Commit message: remake
Parts:
- removed J2: GH125-S06DCA-00, kicad_api_lib:GH125-S06DCA-00, symbol GH125-S06DCA-00:GH125-S06DCA-00
- added J4: GH125-S02CCA-00, kicad_api_lib:GH125-S02CCA-00, symbol GH125-S02CCA-00:GH125-S02CCA-00
- C1, C10, C11, C12, C13, C14, C15, C16, C17, C18, C2, C3, C4, C5, C6, C7, C8, C9, R1, R10, R11, R12, R13, R14, R15, R16, R17, R18, R19, R2, R20, R3, R4, R5, R6, R7, R8, R9: footprint Capacitor_SMD:C_0201_0603Metric -> Capacitor_SMD:C_0603_1608Metric
Connections:
- net +5VIN: now also J4.2
- net AGND: now also J4.1
- net AGND_SHIELD: now also J4.3, J4.4
- net COIL_RAW_N: now also J1.1; no longer J1.2
- net COIL_RAW_P: now also J1.2; no longer J1.1
